File: Hardware/StarNecklace.kicad_pcb (KiCad board)
At the start: 2 copper layers, 55.1 x 54.6 mm, 15 parts, among them J1 Conn_02x03_Odd_Even, SW1 SW_SPDT, U1 ATtiny13A

Commit message: feat: init routing
Parts:
- added G***: LOGO, LOGO, B.Cu at (97.8, 65.0)
- J1: moved to B.Cu
- moved J1 55.1 mm to (100.9, 80.8)
- moved D1 50.2 mm to (97.0, 39.6)
- moved D2 50.2 mm to (74.4, 58.6), turned to 180 degrees
- moved D4 50.2 mm to (84.2, 86.6)
- moved R1 50.2 mm to (96.9, 44.3)
- moved R2 50.2 mm to (79.1, 58.7)
- moved R3 50.2 mm to (115.4, 57.3), turned to 180 degrees
- moved BAT1 50.2 mm to (97.8, 65.0)
- moved D5 50.2 mm to (112.5, 84.6), turned to 180 degrees
- moved R4 50.2 mm to (85.0, 83.1)
- moved R5 50.2 mm to (112.1, 80.7), turned to 180 degrees
- moved SW1 50.2 mm to (97.2, 50.8)
- moved D3 50.2 mm to (120.2, 57.1)
- moved R6 50.0 mm to (97.7, 70.3), turned to 180 degrees
- moved U1 49.8 mm to (97.6, 64.5)
Routing:
- net GNDREF: track 0.00 -> 136.6 mm, vias 0 -> 4
- net MISO: track 0.00 -> 75.8 mm
- net SCK: track 0.00 -> 47.5 mm
- net MOSI: track 0.00 -> 45.7 mm
- net PB4: track 0.00 -> 40.8 mm, vias 0 -> 2
- net VCC: track 0.00 -> 35.6 mm, vias 0 -> 2
- net PB3: track 0.00 -> 27.2 mm
- net Net-(BAT1-+): track 0.00 -> 23.6 mm
- net RST: track 0.00 -> 20.7 mm
- net Net-(D1-K): track 0.00 -> 6.07 mm
- net Net-(D5-K): track 0.00 -> 4.06 mm
- net Net-(D4-K): track 0.00 -> 3.75 mm
- net Net-(D3-K): track 0.00 -> 3.21 mm
- net Net-(D2-K): track 0.00 -> 3.05 mm
Other:
- board text added: "Created by Angelina Tsuboi"
- board text added: "github.com/ANG13T/star_necklace_attiny13_smd"

Commit message: feat: init silk art
Parts:
- added G***: LOGO, LOGO, F.Cu at (98.8, 63.0)
- moved R4 1.61 mm to (85.0, 81.5)
- moved D4 1.12 mm to (84.2, 85.5)
Routing:
- net GNDREF: track 136.6 -> 135.0 mm
- net PB3: track 27.2 -> 26.1 mm
Other:
- board text added: "By Angelina Tsuboi"
- board text added: "angelinatsuboi.com"
- board text removed: "Created by Angelina Tsuboi"
- board text removed: "github.com/ANG13T/star_necklace_attiny13_smd"

Commit message: feat: commit design files
Routing:
- net PB4: track 40.8 -> 42.5 mm
Changed lines of the file:
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@@
       (outputformat 1)
       (mirror false)
-      (drillshape 1)
+      (drillshape 0)
       (scaleselection 1)
-      (outputdirectory "")
+      (outputdirectory "/Users/angelinatsuboi/Desktop/star_necklace_attiny13_smd/Production/")
     )
   )
@@
     (fp_line (start 1 0.625) (end -1 0.625)
       (stroke (width 0.1) (type solid)) (layer "F.Fab"))
-    (pad "1" smd roundrect (at -0.9125 0 180) (size 1.025 1.4) (layers "F.Cu" "F.Paste" "F.Mask") (roundrect_rratio 0.243902)
+    (pad "1" smd roundrect (at -0.9125 0 180) (size 1.025 1.4) (layers "F.Cu" "F.Paste" "F.Mask") (roundrect_rratio 0.243902439)
       (net 6 "Net-(D5-K)") (pintype "passive"))
-    (pad "2" smd roundrect (at 0.9125 0 180) (size 1.025 1.4) (layers "F.Cu" "F.Paste" "F.Mask") (roundrect_rratio 0.243902)
+    (pad "2" smd roundrect (at 0.9125 0 180) (size 1.025 1.4) (layers "F.Cu" "F.Paste" "F.Mask") (roundrect_rratio 0.243902439)
       (net 2 "GNDREF") (pintype "passive"))
     (model "${KICAD6_3DMODEL_DIR}/Resistor_SMD.3dshapes/R_0805_2012Metric.wrl"
@@
     (fp_line (start 1 0.625) (end -1 0.625)
       (stroke (width 0.1) (type solid)) (layer "F.Fab"))
-    (pad "1" smd roundrect (at -0.9125 0 180) (size 1.025 1.4) (layers "F.Cu" "F.Paste" "F.Mask") (roundrect_rratio 0.243902)
+    (pad "1" smd roundrect (at -0.9125 0 180) (size 1.025 1.4) (layers "F.Cu" "F.Paste" "F.Mask") (roundrect_rratio 0.243902439)
       (net 4 "Net-(D3-K)") (pintype "passive"))
-    (pad "2" smd roundrect (at 0.9125 0 180) (size 1.025 1.4) (layers "F.Cu" "F.Paste" "F.Mask") (roundrect_rratio 0.243902)
+    (pad "2" smd roundrect (at 0.9125 0 180) (size 1.025 1.4) (layers "F.Cu" "F.Paste" "F.Mask") (roundrect_rratio 0.243902439)
       (net 2 "GNDREF") (pintype "passive"))
     (model "${KICAD6_3DMODEL_DIR}/Resistor_SMD.3dshapes/R_0805_2012Metric.wrl"
@@
     (fp_line (start 1 0.625) (end -1 0.625)
       (stroke (width 0.1) (type solid)) (layer "F.Fab"))
-    (pad "1" smd roundrect (at -0.9125 0 180) (size 1.025 1.4) (layers "F.Cu" "F.Paste" "F.Mask") (roundrect_rratio 0.243902)
+    (pad "1" smd roundrect (at -0.9125 0 180) (size 1.025 1.4) (layers "F.Cu" "F.Paste" "F.Mask") (roundrect_rratio 0.243902439)
       (net 7 "VCC") (pintype "passive"))
-    (pad "2" smd roundrect (at 0.9125 0 180) (size 1.025 1.4) (layers "F.Cu" "F.Paste" "F.Mask") (roundrect_rratio 0.243902)
+    (pad "2" smd roundrect (at 0.9125 0 180) (size 1.025 1.4) (layers "F.Cu" "F.Paste" "F.Mask") (roundrect_rratio 0.243902439)
       (net 8 "RST") (pintype "passive"))
     (model "${KICAD6_3DMODEL_DIR}/Resistor_SMD.3dshapes/R_0805_2012Metric.wrl"
@@
     (fp_line (start 1 0.625) (end -1 0.625)
       (stroke (width 0.1) (type solid)) (layer "F.Fab"))
-    (pad "1" smd roundrect (at -0.9125 0) (size 1.025 1.4) (layers "F.Cu" "F.Paste" "F.Mask") (roundrect_rratio 0.243902)
+    (pad "1" smd roundrect (at -0.9125 0) (size 1.025 1.4) (layers "F.Cu" "F.Paste" "F.Mask") (roundrect_rratio 0.243902439)
       (net 3 "Net-(D2-K)") (pintype "passive"))
-    (pad "2" smd roundrect (at 0.9125 0) (size 1.025 1.4) (layers "F.Cu" "F.Paste" "F.Mask") (roundrect_rratio 0.243902)
+    (pad "2" smd roundrect (at 0.9125 0) (size 1.025 1.4) (layers "F.Cu" "F.Paste" "F.Mask") (roundrect_rratio 0.243902439)
       (net 2 "GNDREF") (pintype "passive"))
     (model "${KICAD6_3DMODEL_DIR}/Resistor_SMD.3dshapes/R_0805_2012Metric.wrl"
@@
     (fp_line (start 1 0.625) (end -1 0.625)
       (stroke (width 0.1) (type solid)) (layer "F.Fab"))
-    (pad "1" smd roundrect (at -0.9125 0 90) (size 1.025 1.4) (layers "F.Cu" "F.Paste" "F.Mask") (roundrect_rratio 0.243902)
+    (pad "1" smd roundrect (at -0.9125 0 90) (size 1.025 1.4) (layers "F.Cu" "F.Paste" "F.Mask") (roundrect_rratio 0.243902439)
       (net 1 "Net-(D1-K)") (pintype "passive"))
-    (pad "2" smd roundrect (at 0.9125 0 90) (size 1.025 1.4) (layers "F.Cu" "F.Paste" "F.Mask") (roundrect_rratio 0.243902)
+    (pad "2" smd roundrect (at 0.9125 0 90) (size 1.025 1.4) (layers "F.Cu" "F.Paste" "F.Mask") (roundrect_rratio 0.243902439)
       (net 2 "GNDREF") (pintype "passive"))
     (model "${KICAD6_3DMODEL_DIR}/Resistor_SMD.3dshapes/R_0805_2012Metric.wrl"
@@
     (fp_line (start 1 0.625) (end -1 0.625)
       (stroke (width 0.1) (type solid)) (layer "F.Fab"))
-    (pad "1" smd roundrect (at -0.9125 0) (size 1.025 1.4) (layers "F.Cu" "F.Paste" "F.Mask") (roundrect_rratio 0.243902)
+    (pad "1" smd roundrect (at -0.9125 0) (size 1.025 1.4) (layers "F.Cu" "F.Paste" "F.Mask") (roundrect_rratio 0.243902439)
       (net 5 "Net-(D4-K)") (pintype "passive"))
-    (pad "2" smd roundrect (at 0.9125 0) (size 1.025 1.4) (layers "F.Cu" "F.Paste" "F.Mask") (roundrect_rratio 0.243902)
+    (pad "2" smd roundrect (at 0.9125 0) (size 1.025 1.4) (layers "F.Cu" "F.Paste" "F.Mask") (roundrect_rratio 0.243902439)
       (net 2 "GNDREF") (pintype "passive"))
     (model "${KICAD6_3DMODEL_DIR}/Resistor_SMD.3dshapes/R_0805_2012Metric.wrl"
@@
       (stroke (width 0) (type solid)) (fill solid) (layer "B.SilkS"))
   )
+  (gr_circle (center 114.5 84.55) (end 114.525 84.6)
+    (stroke (width 0.1) (type default)) (fill none) (layer "F.SilkS"))
+  (gr_circle (center 82.275 85.5) (end 82.3 85.55)
+    (stroke (width 0.1) (type default)) (fill none) (layer "F.SilkS"))
+  (gr_circle (center 118.325 57.1) (end 118.35 57.15)
+    (stroke (width 0.1) (type default)) (fill none) (layer "F.SilkS"))
+  (gr_circle (center 76.25 58.625) (end 76.275 58.675)
+    (stroke (width 0.1) (type default)) (fill none) (layer "F.SilkS"))
+  (gr_circle (center 93.375 62.575) (end 93.4 62.6)
+    (stroke (width 0.1) (type default)) (fill none) (layer "F.SilkS"))
+  (gr_circle (center 94.975 39.65) (end 95 39.7)
+    (stroke (width 0.1) (type default)) (fill none) (layer "F.SilkS"))
   (gr_curve (pts (xy 81.666391 90.178892) (xy 80.019391 89.054542) (xy 81.833291 73.635178) (xy 81.144825 71.73209))
     (stroke (width 0.05) (type solid)) (layer "Edge.Cuts"))
@@
   (segment (start 85.0375 85.25) (end 85.0375 73.611104) (width 0.2) (layer "F.Cu") (net 9))
   (segment (start 111.6945 84.6338) (end 110.2662 84.6338) (width 0.2) (layer "F.Cu") (net 10))
-  (segment (start 95.151004 65.1774) (end 95.4924 65.1774) (width 0.2) (layer "F.Cu") (net 10))
+  (segment (start 94.03689 65.1774) (end 95.4924 65.1774) (width 0.2) (layer "F.Cu") (net 10))
+  (segment (start 88.85 70.36429) (end 94.05429 65.16) (width 0.2) (layer "F.Cu") (net 10))
   (segment (start 110.2338 84.6338) (end 110.2162 84.6338) (width 0.2) (layer "F.Cu") (net 10))
   (segment (start 110.2162 84.6338) (end 110.2 84.65) (width 0.2) (layer "F.Cu") (net 10))
-  (segment (start 88.85 76.85) (end 88.85 71.478404) (width 0.2) (layer "F.Cu") (net 10))
-  (segment (start 88.85 71.478404) (end 95.151004 65.1774) (width 0.2) (layer "F.Cu") (net 10))
+  (segment (start 94.05429 65.16) (end 95.1 65.16) (width 0.2) (layer "F.Cu") (net 10))
+  (segment (start 88.85 76.85) (end 88.85 70.36429) (width 0.2) (layer "F.Cu") (net 10))
   (segment (start 110.25 84.65) (end 110.2338 84.6338) (width 0.2) (layer "F.Cu") (net 10))
   (segment (start 110.2662 84.6338) (end 110.25 84.65) (width 0.2) (layer "F.Cu") (net 10))
