File: Hardware/StarNecklace.kicad_sch (KiCad schematic)
At the start: 14 parts, among them J1 Conn_02x03_Odd_Even, SW1 SW_SPDT, U1 ATtiny13A

Commit message: feat: init schematic
Parts:
- added R6: 4.7k, Resistor_SMD:R_0805_2012Metric, symbol Device:R_US
- J1: footprint (none) -> Connector_PinHeader_2.54mm:PinHeader_2x03_P2.54mm_Vertical
Connections:
- net RST: now also R6.2
- net VCC: now also R6.1
Changed lines of the file:
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@@
+    )
+  )
+  (global_label "RST" (shape input) (at 78.74 51.435 270) (fields_autoplaced)
+    (effects (font (size 1.27 1.27)) (justify right))
+    (property "Intersheetrefs" "${INTERSHEET_REFS}" (at 78.74 57.8673 90)
+      (effects (font (size 1.27 1.27)) (justify right) hide)
     )
   )
@@
     )
   )
+  (symbol (lib_id "Device:R_US") (at 78.74 47.625 0) (unit 1)
+    (in_bom yes) (on_board yes) (dnp no) (fields_autoplaced)
+    (property "Reference" "R6" (at 81.28 46.355 0)
+      (effects (font (size 1.27 1.27)) (justify left))
+    )
+    (property "Value" "4.7k" (at 81.28 48.895 0)
+      (effects (font (size 1.27 1.27)) (justify left))
+    )
+    (property "Footprint" "Resistor_SMD:R_0805_2012Metric" (at 79.756 47.879 90)
+      (effects (font (size 1.27 1.27)) hide)
+    )
+    (property "Datasheet" "~" (at 78.74 47.625 0)
+      (effects (font (size 1.27 1.27)) hide)
+    )
+    (pin "1")
+    (pin "2")
+    (instances
+      (project "StarNecklace"
+        (path "/5df35fb8-dff4-4661-b07b-6cca2458bfeb"
+          (reference "R6") (unit 1)
+        )
+      )
+    )
+  )
   (symbol (lib_id "power:GNDREF") (at 120.65 62.23 0) (unit 1)
     (in_bom yes) (on_board yes) (dnp no) (fields_autoplaced)
@@
       (effects (font (size 1.27 1.27)) hide)
     )
-    (property "Footprint" "" (at 128.27 81.28 0)
+    (property "Footprint" "Connector_PinHeader_2.54mm:PinHeader_2x03_P2.54mm_Vertical" (at 128.27 81.28 0)
       (effects (font (size 1.27 1.27)) hide)
     )
@@
         )
       )
+    )
+  )
+  (symbol (lib_id "power:VCC") (at 78.74 43.815 0) (unit 1)
+    (in_bom yes) (on_board yes) (dnp no) (fields_autoplaced)
+    (property "Reference" "#PWR08" (at 78.74 47.625 0)
+      (effects (font (size 1.27 1.27)) hide)
+    )
+    (property "Value" "VCC" (at 78.74 40.005 0)
+      (effects (font (size 1.27 1.27)))
+    )
+    (property "Footprint" "" (at 78.74 43.815 0)
+      (effects (font (size 1.27 1.27)) hide)
+    )
+    (property "Datasheet" "" (at 78.74 43.815 0)
+      (effects (font (size 1.27 1.27)) hide)
+    )
+    (pin "1")
+    (instances
+      (project "StarNecklace"
+        (path "/5df35fb8-dff4-4661-b07b-6cca2458bfeb"
+          (reference "#PWR08") (unit 1)
+        )
+      )

Commit message: feat: update footprints and init pcb
Parts:
- BAT1: footprint Battery:BatteryHolder_Keystone_1058_1x2032 -> Battery:BatteryHolder_Keystone_1060_1x2032
- SW1: footprint SW SS12D:Schiebeschalter SS-12D00.kicad_mod -> Button_Switch_THT:Schiebeschalter_SS-12D00
Changed lines of the file:
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@@
       (effects (font (size 1.27 1.27)) hide)
     )
-    (property "Footprint" "SW SS12D:Schiebeschalter SS-12D00.kicad_mod" (at 63.5 82.55 0)
+    (property "Footprint" "Button_Switch_THT:Schiebeschalter_SS-12D00" (at 63.5 82.55 0)
       (effects (font (size 1.27 1.27)) hide)
     )
@@
       (effects (font (size 1.27 1.27)))
     )
-    (property "Footprint" "Battery:BatteryHolder_Keystone_1058_1x2032" (at 81.026 85.09 90)
-      (effects (font (size 1.27 1.27)) hide)
-    )
+    (property "Footprint" "Battery:BatteryHolder_Keystone_1060_1x2032" (at 81.026 85.09 90)
+      (effects (font (size 1.27 1.27)) hide)
+    )
